Commit message: v3: First underwater dynamics prototype
- Added custom buoyancy plugin
- Added quadratic drag plugin
- Added tail thrust plugin
- Implemented fish teleoperation
- Integrated ros2_control controllers
- Tuned neutral buoyancy
- Stable articulated fish simulation
- Prepared architecture for distributed hydrodynamics

File: src/fishbot_description/urdf/fishbot.urdf.xacro (robot description, xacro)
@@ -22,12 +22,12 @@
     <inertial>
       <origin xyz="0 0 0" rpy="0 0 0"/>
-      <mass value="1.0"/>
-      <inertia
-        ixx="0.01"
-        ixy="0"
-        ixz="0"
-        iyy="0.01"
-        iyz="0"
-        izz="0.01"/>
+      <mass value="4.00"/>
+      <inertia
+          ixx="0.01208"
+          ixy="0"
+          ixz="0"
+          iyy="0.03333"
+          iyz="0"
+          izz="0.03750"/>
     </inertial>
   </link>
@@ -56,12 +56,12 @@
       <origin xyz="-0.06 0 0"
               rpy="0 0 0"/>
-      <mass value="0.2"/>
-      <inertia
-        ixx="0.001"
-        ixy="0"
-        ixz="0"
-        iyy="0.001"
-        iyz="0"
-        izz="0.001"/>
+      <mass value="0.15"/>
+      <inertia
+          ixx="0.000216"
+          ixy="0"
+          ixz="0"
+          iyy="0.000130"
+          iyz="0"
+          izz="0.000336"/>
     </inertial>
   </link>
@@ -104,13 +104,13 @@
       <origin xyz="0 0.03 0"
               rpy="0 0 0"/>
-      <mass value="0.05"/>
-      <inertia
-        ixx="0.0001"
-        ixy="0"
-        ixz="0"
-        iyy="0.0001"
-        iyz="0"
-        izz="0.0001"/>
-    </inertial>
+      <mass value="0.03"/>
+      <inertia
+          ixx="0.0000097"
+          ixy="0"
+          ixz="0"
+          iyy="0.0000128"
+          iyz="0"
+          izz="0.0000213"/>
+      </inertial>
   </link>
   <!-- Left Fin Joint -->
@@ -152,13 +152,13 @@
       <origin xyz="0 -0.03 0"
               rpy="0 0 0"/>
-      <mass value="0.05"/>
-      <inertia
-        ixx="0.0001"
-        ixy="0"
-        ixz="0"
-        iyy="0.0001"
-        iyz="0"
-        izz="0.0001"/>
-    </inertial>
+      <mass value="0.03"/>
+      <inertia
+          ixx="0.0000097"
+          ixy="0"
+          ixz="0"
+          iyy="0.0000128"
+          iyz="0"
+          izz="0.0000213"/>
+      </inertial>
   </link>
   <!-- Right Fin Joint -->
@@ -216,3 +216,21 @@
   </plugin>
 </gazebo>
+<gazebo>
+  <plugin
+      name="fishbot_buoyancy"
+      filename="libbuoyancy_plugin.so">
+  </plugin>
+</gazebo>
+<gazebo>
+  <plugin
+      name="fishbot_drag"
+      filename="libdrag_plugin.so">
+  </plugin>
+</gazebo>
+<gazebo>
+  <plugin
+      name="fishbot_thrust"
+      filename="libthrust_plugin.so">
+  </plugin>
+</gazebo>
 </robot>
