Commit message: Working Gravity, Buoyancy, Drag, Thrust and Teleop

File: src/fishbot_description/urdf/fishbot.urdf.xacro (robot description, xacro)
@@ -22,12 +22,12 @@
     <inertial>
       <origin xyz="0 0 0" rpy="0 0 0"/>
-      <mass value="4.00"/>
-      <inertia
-          ixx="0.01208"
-          ixy="0"
-          ixz="0"
-          iyy="0.03333"
-          iyz="0"
-          izz="0.03750"/>
+      <mass value="3.31"/>
+      <inertia
+      ixx="0.01034"
+      ixy="0.0"
+      ixz="0.0"
+      iyy="0.02758"
+      iyz="0.0"
+      izz="0.03172"/>
     </inertial>
   </link>
@@ -56,12 +56,12 @@
       <origin xyz="-0.06 0 0"
               rpy="0 0 0"/>
-      <mass value="0.15"/>
-      <inertia
-          ixx="0.000216"
-          ixy="0"
-          ixz="0"
-          iyy="0.000130"
-          iyz="0"
-          izz="0.000336"/>
+      <mass value="0.66"/>
+      <inertia
+        ixx="0.00095"
+        ixy="0.0"
+        ixz="0.0"
+        iyy="0.00057"
+        iyz="0.0"
+        izz="0.00148"/>
     </inertial>
   </link>
@@ -104,13 +104,13 @@
       <origin xyz="0 0.03 0"
               rpy="0 0 0"/>
-      <mass value="0.03"/>
-      <inertia
-          ixx="0.0000097"
-          ixy="0"
-          ixz="0"
-          iyy="0.0000128"
-          iyz="0"
-          izz="0.0000213"/>
-      </inertial>
+      <mass value="0.165"/>
+      <inertia
+        ixx="0.000053"
+        ixy="0.0"
+        ixz="0.0"
+        iyy="0.000070"
+        iyz="0.0"
+        izz="0.000117"/>
+    </inertial>
   </link>
   <!-- Left Fin Joint -->
@@ -152,13 +152,13 @@
       <origin xyz="0 -0.03 0"
               rpy="0 0 0"/>
-      <mass value="0.03"/>
-      <inertia
-          ixx="0.0000097"
-          ixy="0"
-          ixz="0"
-          iyy="0.0000128"
-          iyz="0"
-          izz="0.0000213"/>
-      </inertial>
+      <mass value="0.165"/>
+      <inertia
+        ixx="0.000053"
+        ixy="0.0"
+        ixz="0.0"
+        iyy="0.000070"
+        iyz="0.0"
+        izz="0.000117"/>
+    </inertial>
   </link>
   <!-- Right Fin Joint -->
@@ -232,4 +232,16 @@
       name="fishbot_thrust"
       filename="libthrust_plugin.so">
+    <thrust_coefficient>0.5</thrust_coefficient>
+    <steering_coefficient>0.5</steering_coefficient>
+    <velocity_filter_alpha>0.9</velocity_filter_alpha>
+    <water_density>1000.0</water_density>
+    <tail_area>0.013</tail_area>
+    <tail_lever_length>0.06</tail_lever_length>
+  </plugin>
+</gazebo>
+<gazebo>
+  <plugin
+      name="fishbot_fin_hydrodynamics"
+      filename="libfin_hydrodynamics_plugin.so">
   </plugin>
 </gazebo>

Commit message: Replaced primitive model with Fusion360 CAD meshes

File: src/fishbot_description/urdf/fishbot.urdf.xacro (robot description, xacro)
@@ -6,7 +6,8 @@
   <link name="base_link">
     <visual>
-      <origin xyz="0 0 0" rpy="0 0 0"/>
-      <geometry>
-        <box size="0.3 0.15 0.1"/>
+      <origin xyz="0 0 0" rpy="3.1416 0 -1.5708"/>
+      <geometry>
+        <mesh filename="src/fishbot_description/meshes/base_link.stl"
+        scale="0.001 0.001 0.001"/>
       </geometry>
       <material name="blue">
@@ -15,11 +16,12 @@
     </visual>
     <collision>
-      <origin xyz="0 0 0" rpy="0 0 0"/>
-      <geometry>
-        <box size="0.3 0.15 0.1"/>
-      </geometry>
-    </collision>
-    <inertial>
-      <origin xyz="0 0 0" rpy="0 0 0"/>
+      <origin xyz="0 0 0" rpy="0 0 1.5708"/>
+      <geometry>
+        <mesh filename="src/fishbot_description/meshes/base_link.stl"
+        scale="0.001 0.001 0.001"/>
+      </geometry>
+    </collision>
+    <inertial>
+      <origin xyz="0 0 0" rpy="0 0 1.5708"/>
       <mass value="3.31"/>
       <inertia
@@ -37,18 +39,20 @@
   <link name="tail_link">
     <visual>
+      <origin xyz="0 0 0"
+              rpy="3.1416 3.1416 4.7124"/>
+      <geometry>
+        <mesh filename="src/fishbot_description/meshes/tail_link.stl"
+        scale="0.001 0.001 0.001"/>
+      </geometry>
+      <material name="red">
+        <color rgba="1 0.3 0.3 1"/>
+      </material>
+    </visual>
+    <collision>
       <origin xyz="-0.06 0 0"
               rpy="1.5708 1.5708 0"/>
       <geometry>
-        <box size="0.10 0.13 0.02"/>
-      </geometry>
-      <material name="red">
-        <color rgba="1 0.3 0.3 1"/>
-      </material>
-    </visual>
-    <collision>
-      <origin xyz="-0.06 0 0"
-              rpy="1.5708 1.5708 0"/>
-      <geometry>
-        <box size="0.10 0.13 0.02"/>
+        <mesh filename="src/fishbot_description/meshes/tail_link.stl"
+        scale="0.001 0.001 0.001"/>
       </geometry>
     </collision>
@@ -68,5 +72,5 @@
   <!-- Tail Joint -->
   <joint name="tail_joint" type="revolute">
-    <origin xyz="-0.15 0 0"
+    <origin xyz="-0.065 0 0"
             rpy="0 0 0"/>
     <parent link="base_link"/>
@@ -85,8 +89,9 @@
   <link name="left_fin_link">
     <visual>
-      <origin xyz="0 0.03 0"
-              rpy="0 0 0"/>
-      <geometry>
-        <box size="0.07 0.06 0.015"/>
+      <origin xyz="0 -0.07 0"
+              rpy="0 0 1.5708"/>
+      <geometry>
+        <mesh filename="src/fishbot_description/meshes/left_fin_link.stl"
+        scale="0.001 0.001 0.001"/>
       </geometry>
       <material name="light_blue">
@@ -98,5 +103,6 @@
               rpy="0 0 0"/>
       <geometry>
-        <box size="0.07 0.06 0.015"/>
+        <mesh filename="src/fishbot_description/meshes/left_fin_link.stl"
+        scale="0.001 0.001 0.001"/>
       </geometry>
     </collision>
@@ -133,8 +139,9 @@
   <link name="right_fin_link">
     <visual>
-      <origin xyz="0 -0.03 0"
-              rpy="0 0 0"/>
-      <geometry>
-        <box size="0.07 0.06 0.015"/>
+      <origin xyz="0 0.07 0"
+              rpy="0 0 1.5708"/>
+      <geometry>
+        <mesh filename="src/fishbot_description/meshes/right_fin_link.stl"
+        scale="0.001 0.001 0.001"/>
       </geometry>
       <material name="light_blue">
@@ -146,5 +153,6 @@
               rpy="0 0 0"/>
       <geometry>
-        <box size="0.07 0.06 0.015"/>
+        <mesh filename="src/fishbot_description/meshes/right_fin_link.stl"
+        scale="0.001 0.001 0.001"/>
       </geometry>
     </collision>
